File: pcbs/street_sense_cpu/street_sense_cpu.sch (KiCad schematic (older format))
At the start: 20 parts, among them J1 Conn_01x08, J10 Conn_01x06, J11 Conn_01x09, J13 Conn_01x02, J14 Conn_01x02, J3 Conn_01x06, J4 Conn_01x04, J5 Conn_01x02, J6 Conn_01x02, J7 Conn_01x08, J9 Conn_01x02, U1 Lolin_D32_Pro, U2 DS3231_Module

Commit message: updated CPU schematic
Parts:
- added TP3, TP4: TestPoint, TestPoint:TestPoint_Loop_D2.50mm_Drill1.0mm, symbol Connector:TestPoint
- JP1, JP2: footprint Jumper:SolderJumper-2_P1.3mm_Open_Pad1.0x1.5mm -> street_sense_footprints:SolderJumper-2_P1.3mm_Open_Pad1.0x1.5mm
- R2: value 470k -> 68k
- renumbered J7 to J1, J13 to J10, J14 to J11, J9 to J2, J1 to J3, J3 to J4, J4 to J5, J5 to J6, J6 to J7, J10 to J8, J11 to J9, R7 to R3
Connections:
- net +3V3: now also J1.2 (Pin_2), TP3.1; no longer J1.4 (Pin_4)
- net BAT: now also J1.7 (Pin_7); no longer J1.2 (Pin_2)
- net DRDY: now also J1.1 (Pin_1); no longer J1.5 (Pin_5)
- net GND: now also J1.8 (Pin_8), TP4.1; no longer J1.1 (Pin_1), J1.6 (Pin_6)
- net SCK: no longer J4.1 (Pin_1), U1.13 (GPIO13)
- net SCL: now also J1.5 (Pin_5); no longer J1.7 (Pin_7)
- net SDA: now also J1.6 (Pin_6); no longer J1.8 (Pin_8)
- net USB: no longer TP1.1
- net at J5.1 (Pin_1), JP1.1: now also TP1.1
- net at JP2.1: now also J5.3 (Pin_3); no longer J5.2 (Pin_2)
- net at J6.1 (Pin_1): now also J5.2 (Pin_2); no longer J5.3 (Pin_3)
- net SD renamed M_SD
- net WS renamed M_WS
- new net M_SCK: J4.1 (Pin_1), U1.13 (GPIO13)
- no-connect marks 10 -> 11
Other:
- moved on the sheet: JP1, TP1, U2
